Commit message: change urdf

File: diana7_dual_dexh13_description/urdf/dual_diana7_dexh13.urdf (robot description, URDF)
Before this commit: robot dual_diana7_dexh13, 2368 links, 2367 joints
Joints:
- joint left_dexh13_flange_to_palm_joint: origin xyz=0 0 0.0863588256836 rpy=0 -1.57079632679 0 -> xyz=0.028555454 0.042861867 0.067315626 rpy=-2.671200996 -1.432453113 1.125485105
- joint left_sensor_to_dexh13_flange_joint: origin xyz=0 0 0.046 rpy=0 0 -0.436332313817 -> xyz=-0.043 0.013 0.042 rpy=1.564269285 0.016179064 0.462469649
- joint right_dexh13_flange_to_palm_joint: origin xyz=0 0 0.0863588256836 rpy=0 -1.57079632679 0 -> xyz=-0.00188914404 0.00299943662 0.06653594754 rpy=2.92260538187 -1.57079544121 1.78978734387
- joint right_sensor_to_dexh13_flange_joint: origin xyz=0 0 0.046 rpy=0 0 -2.00712864061 -> xyz=0.014 -0.02846 0.074 rpy=1.57078802587 0.00000586142 -2.68779868756

Commit message: Add FreeCAD MCP setup and tactile experiment assets

File: diana7_dual_dexh13_description/urdf/dual_diana7_dexh13.urdf (robot description, URDF)
Before this commit: robot dual_diana7_dexh13, 2368 links, 2367 joints
Joints:
- joint left_dexh13_flange_to_palm_joint: origin xyz=0.028555454 0.042861867 0.067315626 rpy=-2.671200996 -1.432453113 1.125485105 -> xyz=-0.00294541425 0.01036186700 0.06731562602 rpy=-2.671200996 -1.432453113 1.125485105
- joint left_sensor_to_dexh13_flange_joint: origin xyz=-0.043 0.013 0.042 rpy=1.564269285 0.016179064 0.462469649 -> xyz=-0.01443597095 0.02747700630 0.07398542195 rpy=1.564269285 0.016179064 0.462469649

Commit message: Align right DexH13 flange and palm from FreeCAD reference

File: diana7_dual_dexh13_description/urdf/dual_diana7_dexh13.urdf (robot description, URDF)
Before this commit: robot dual_diana7_dexh13, 2368 links, 2367 joints
Joints:
- joint right_dexh13_flange_to_palm_joint: origin xyz=-0.00188914404 0.00299943662 0.06653594754 rpy=2.92260538187 -1.57079544121 1.78978734387 -> xyz=-0.00019594765 0.00749938129 0.06908118221 rpy=0 -1.5707963267949 -1.5707963267949
